File: Trasncan-Panda-Carrier-Board/Carrier Board.brd (EAGLE design)
At the start: 90 x 38.6 mm, 57 parts, among them J1 B2B-PH-SM4-TB(LF)(SN), J2 B2B-PH-SM4-TB(LF)(SN), J3 BM04B-SRSS-TBT(LF)(SN), J4 BM06B-SRSS-TBT(LF)(SN), J5 BM06B-SRSS-TBT(LF)(SN), J6 BM06B-SRSS-TBT(LF)(SN), J7 BM04B-SRSS-TBT(LF)(SN), J8 BM04B-SRSS-TBT(LF)(SN), J9 BM04B-SRSS-TBT(LF)(SN), P1 Particle Boron / Xenon / Argon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

Commit message: Rectangular Sensor Board
Parts:
- removed FRAME1, FRAME2, FRAME3: FRAME-LETTER, SparkFun-Aesthetics:CREATIVE_COMMONS
Changed lines of the file:
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@@
 <layer number="29" name="tStop" color="7" fill="3" visible="yes" active="yes"/>
 <layer number="30" name="bStop" color="7" fill="6" visible="no" active="yes"/>
-<layer number="31" name="tCream" color="7" fill="4" visible="yes" active="yes"/>
+<layer number="31" name="tCream" color="7" fill="4" visible="no" active="yes"/>
 <layer number="32" name="bCream" color="7" fill="5" visible="no" active="yes"/>
 <layer number="33" name="tFinish" color="6" fill="3" visible="no" active="yes"/>
@@
 <layer number="37" name="tTest" color="7" fill="1" visible="no" active="yes"/>
 <layer number="38" name="bTest" color="7" fill="1" visible="no" active="yes"/>
-<layer number="39" name="tKeepout" color="4" fill="11" visible="yes" active="yes"/>
+<layer number="39" name="tKeepout" color="4" fill="11" visible="no" active="yes"/>
 <layer number="40" name="bKeepout" color="1" fill="11" visible="no" active="yes"/>
 <layer number="41" name="tRestrict" color="4" fill="10" visible="no" active="yes"/>
@@
 <layer number="49" name="Reference" color="7" fill="1" visible="no" active="yes"/>
 <layer number="50" name="dxf" color="7" fill="1" visible="no" active="no"/>
-<layer number="51" name="tDocu" color="7" fill="1" visible="no" active="yes"/>
+<layer number="51" name="tDocu" color="7" fill="1" visible="yes" active="yes"/>
 <layer number="52" name="bDocu" color="7" fill="1" visible="no" active="yes"/>
 <layer number="53" name="tGND_GNDA" color="7" fill="9" visible="no" active="no"/>
@@
 <attribute name="POPULATE" value="0" x="86.1568" y="11.557" size="1.778" layer="28" rot="MR90" display="off"/>
 </element>
-<element name="FRAME1" library="SparkFun-Aesthetics" library_urn="urn:adsk.eagle:library:507" package="CREATIVE_COMMONS" package3d_urn="urn:adsk.eagle:package:37121/1" value="FRAME-LETTER" x="0.0254" y="-11.811" smashed="yes">
-<attribute name="POPULATE" value="0" x="0.0254" y="-11.811" size="1.778" layer="27" display="off"/>
-</element>
-<element name="FRAME2" library="SparkFun-Aesthetics" library_urn="urn:adsk.eagle:library:507" package="CREATIVE_COMMONS" package3d_urn="urn:adsk.eagle:package:37121/1" value="FRAME-LETTER" x="-0.0254" y="-7.9756" smashed="yes">
-<attribute name="POPULATE" value="0" x="-0.0254" y="-7.9756" size="1.778" layer="27" display="off"/>
-</element>
 <element name="R7" library="Custom Components" package="0805" package3d_urn="urn:adsk.eagle:package:39651/1" value="10k" x="64.008" y="9.906" smashed="yes">
 <attribute name="HOUSEPART" value="YES" x="64.008" y="9.906" size="1.778" layer="27" display="off"/>
@@
 <attribute name="URL" value="https://factory.macrofab.com/part/MF-CAP-0805-0.1uF" x="79.756" y="18.796" size="1.778" layer="27" display="off"/>
 <attribute name="VALUE" value="0.1uF" x="79.756" y="18.796" size="1.778" layer="27" display="off"/>
-</element>
-<element name="FRAME3" library="SparkFun-Aesthetics" library_urn="urn:adsk.eagle:library:507" package="CREATIVE_COMMONS" package3d_urn="urn:adsk.eagle:package:37121/1" value="FRAME-LETTER" x="90.424" y="19.2786" smashed="yes">
-<attribute name="POPULATE" value="0" x="90.424" y="19.2786" size="1.778" layer="27" display="off"/>
 </element>
 <element name="JP7" library="SparkFun-Jumpers" library_urn="urn:adsk.eagle:library:528" package="SMT-JUMPER_2_NO_SILK" package3d_urn="urn:adsk.eagle:package:39279/1" value="JUMPER-SMT_2_NO_SILK" x="73.66" y="21.082" smashed="yes" rot="MR270">
@@
 <contactref element="C2" pad="2"/>
 <polygon width="0.254" layer="1" rank="2">
-<vertex x="-3.7846" y="42.6873875"/>
-<vertex x="99.752840625" y="42.882784375"/>
-<vertex x="99.692475" y="-4.021"/>
-<vertex x="-3.7846" y="-4.2164"/>
+<vertex x="-0.4826" y="39.147684375"/>
+<vertex x="90.092003125" y="39.31861875"/>
+<vertex x="90.040453125" y="-0.735309375"/>
+<vertex x="-0.4826" y="-0.906246875"/>
 </polygon>
 <polygon width="0.254" layer="16">
-<vertex x="-3.595303125" y="47.033259375"/>
-<vertex x="95.4937375" y="46.87546875"/>
-<vertex x="95.27434375" y="-3.176103125"/>
-<vertex x="-3.376025" y="-3.149821875"/>
+<vertex x="-0.54838125" y="39.40598125"/>
+<vertex x="90.115228125" y="39.26160625"/>
+<vertex x="89.939234375" y="-0.888884375"/>
+<vertex x="-0.372415625" y="-0.864825"/>
 </polygon>
 <contactref element="V1" pad="1"/>
